File: Hardware/CAD/Nachtlicht/Tiny13-Nachtlicht.sch (KiCad schematic (older format))
At the start: 9 parts, among them J1 AVR-ISP-6, J2 Pin 1x3, U3 ATtiny13A-SSU

Commit message: Fix value of R1 to match the one actually used.
Add PDF of schematics, and archive of entire Kicad project.
Parts:
- R1: value 100 Ω -> 27 Ω
Other:
- note added: "(Steckverbinder nicht bestückt.)"
Changed lines of the file:
@@
 EESchema Schematic File Version 4
+LIBS:Tiny13-Nachtlicht-cache
 EELAYER 26 0
 EELAYER END
@@
 encoding utf-8
 Sheet 1 1
-Title ""
-Date ""
-Rev ""
-Comp ""
+Title "Nachtlicht"
+Date "2019-11-22"
+Rev "1.0"
+Comp "DARC OV \"Pentacon Dresden\""
 Comment1 ""
 Comment2 ""
@@
 P 6200 3600
 F 0 "C2" H 6315 3646 50  0000 L CNN
-F 1 "100 nF" H 6315 3555 50  0000 L CNN
+F 1 "100 nF" V 6350 3250 50  0000 L CNN
 F 2 "Capacitors_SMD:C_0805_HandSoldering" H 6238 3450 50  0001 C CNN
 F 3 "~" H 6200 3600 50  0001 C CNN
@@
 U 1 1 5DBCC2B5
 P 6600 3650
-F 0 "D1" V 6504 3808 50  0000 L CNN
-F 1 "PD333-3C/H0/L2" V 6595 3808 50  0000 L CNN
+F 0 "D1" V 6350 3700 50  0000 L CNN
+F 1 "PD333-3C/H0/L2" H 6400 3900 50  0000 L CNN
 F 2 "LEDs:LED-5MM" H 6550 3650 50  0001 C CNN
 F 3 "~" H 6550 3650 50  0001 C CNN
@@
 P 7000 3300
 F 0 "R1" V 6793 3300 50  0000 C CNN
-F 1 "100 Ω" V 6884 3300 50  0000 C CNN
+F 1 "27 Ω" V 6884 3300 50  0000 C CNN
 F 2 "Resistors_SMD:R_0805_HandSoldering" V 6930 3300 50  0001 C CNN
 F 3 "~" H 7000 3300 50  0001 C CNN
@@
 Text Notes 6500 2900 0    50   ~ 0
 Jumper
+Text Notes 5400 5700 0    50   ~ 0
+(Steckverbinder nicht bestückt.)
 $EndSCHEMATC
